File: right-main/right-main.kicad_pcb (KiCad board)
At the start: 2 copper layers, 150.4 x 123.8 mm, 208 parts, among them J1 USBCONN, P1 CONN_4, P2 CONN_5, P3 CONN_6, SW1 PTS525SM10, SW11 SPST, SW12 SPST, SW13 SPST, SW14 SPST, SW15 SPST, SW16 SPST, SW17 SPST, SW21 SPST, SW22 SPST, SW23 SPST, SW24 SPST, SW25 SPST, SW26 SPST, SW27 SPST, SW31 SPST, SW32 SPST, SW33 SPST, SW34 SPST, SW35 SPST, SW36 SPST, SW37 SPST, SW41 SPST, SW42 SPST, SW43 SPST, SW44 SPST, SW45 SPST, SW46 SPST, SW47 SPST, SW52 SPST, SW53 SPST, SW54 SPST, SW55 SPST, SW56 SPST, SW57 SPST, U1 ATMEGA32U4, U2 CAT24C256, X1 16Mhz

Commit message: switch 21
Parts:
- SW21: footprint UGL:Cherry_MX -> ugl:Cherry-MX-Matias-Hybrid
- moved via 38/22mil 0.92 mm to (139.7, 80.8)
Routing:
- net /ROW2: track 158.6 -> 160.6 mm
Changed lines of the file:
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@@
 (kicad_pcb (version 4) (host pcbnew 4.0.1-stable)
   (general
-    (links 323)
+    (links 325)
     (no_connects 0)
     (area 19.803 18.9051 270.000001 165.000001)
     (thickness 1.6)
     (drawings 354)
-    (tracks 951)
+    (tracks 956)
     (zones 0)
     (modules 208)
@@
     (34 B.Paste user)
     (35 F.Paste user)
-    (36 B.SilkS user)
-    (37 F.SilkS user)
+    (36 B.SilkS user hide)
+    (37 F.SilkS user hide)
     (38 B.Mask user)
     (39 F.Mask user)
@@
   )
   (module UGL:via_38_22mil (layer F.Cu)
-    (at 139.8016 81.6864)
+    (at 139.7 80.772)
     (fp_text reference "via 38/22mil" (at 0 -1.8) (layer F.SilkS) hide
       (effects (font (size 0.75 0.75) (thickness 0.15)))
@@
       (net 17 /ROW2))
   )
-  (module UGL:Cherry_MX locked (layer F.Cu)
-    (at 135.2 82.7 180)
-    (fp_text reference SW21 (at 0 4.9 180) (layer F.SilkS)
-      (effects (font (size 1.5 1.5) (thickness 0.3)))
-    )
-    (fp_text value SPST (at 0 0 180) (layer F.SilkS) hide
-      (effects (font (size 1.5 1.5) (thickness 0.3)))
-    )
-    (fp_line (start -7.6 -7.6) (end -7.6 7.6) (layer B.SilkS) (width 0.15))
-    (fp_line (start -7.6 7.6) (end 7.6 7.6) (layer B.SilkS) (width 0.15))
-    (fp_line (start 7.6 -7.6) (end 7.6 7.6) (layer B.SilkS) (width 0.15))
-    (fp_line (start -7.6 -7.6) (end 7.6 -7.6) (layer B.SilkS) (width 0.15))
-    (fp_line (start -7.62 -7.62) (end 7.62 -7.62) (layer F.SilkS) (width 0.15))
-    (fp_line (start 7.62 -7.62) (end 7.62 7.62) (layer F.SilkS) (width 0.15))
-    (fp_line (start 7.62 7.62) (end -7.62 7.62) (layer F.SilkS) (width 0.15))
-    (fp_line (start -7.62 7.62) (end -7.62 -7.62) (layer F.SilkS) (width 0.15))
-    (pad "" np_thru_hole circle (at 0 0 180) (size 4 4) (drill 4) (layers *.Cu *.Mask F.SilkS))
-    (pad 2 thru_hole circle (at -3.81 -2.54 180) (size 2.5 2.5) (drill 1.5) (layers *.Cu *.Mask F.SilkS)
-      (net 17 /ROW2))
-    (pad 1 thru_hole circle (at 2.54 -5.08 180) (size 2.5 2.5) (drill 1.5) (layers *.Cu *.Mask F.SilkS)
-      (net 37 "Net-(D21-Pad2)"))
-  )
   (module UGL:UX60-MB-5S8 locked (layer F.Cu)
     (at 175.849803 43.601924 85.4)
@@
     )
   )
+  (module ugl:Cherry-MX-Matias-Hybrid locked (layer F.Cu)
+    (at 135.2 82.7 180)
+    (tags switch)
+    (fp_text reference SW21 (at 0 3.81 180) (layer F.SilkS)
+      (effects (font (thickness 0.3048)))
+    )
+    (fp_text value SPST (at 0 0 180) (layer F.SilkS) hide
+      (effects (font (thickness 0.3048)))
+    )
+    (fp_line (start -7.62 7.62) (end -7.62 -7.62) (layer B.SilkS) (width 0.15))
+    (fp_line (start 7.62 7.62) (end -7.62 7.62) (layer B.SilkS) (width 0.15))
+    (fp_line (start 7.62 -7.62) (end 7.62 7.62) (layer B.SilkS) (width 0.15))
+    (fp_line (start -7.62 -7.62) (end 7.62 -7.62) (layer B.SilkS) (width 0.15))
+    (fp_line (start -7.75 -6.4) (end -7.75 6.4) (layer F.SilkS) (width 0.15))
+    (fp_line (start 7.75 -6.4) (end 7.75 6.4) (layer F.SilkS) (width 0.15))
+    (fp_line (start -7.75 6.4) (end 7.75 6.4) (layer F.SilkS) (width 0.15))
+    (fp_line (start -7.75 -6.4) (end 7.75 -6.4) (layer F.SilkS) (width 0.15))
+    (fp_line (start -7.62 -7.62) (end 7.62 -7.62) (layer F.SilkS) (width 0.15))
+    (fp_line (start 7.62 -7.62) (end 7.62 7.62) (layer F.SilkS) (width 0.15))
+    (fp_line (start 7.62 7.62) (end -7.62 7.62) (layer F.SilkS) (width 0.15))
+    (fp_line (start -7.62 7.62) (end -7.62 -7.62) (layer F.SilkS) (width 0.15))
+    (pad 0 thru_hole circle (at 0 0 180) (size 3.98018 3.98018) (drill 3.98018) (layers *.Cu *.Mask F.SilkS))
+    (pad 1 thru_hole circle (at 2.54 -5.08 180) (size 2.6 2.6) (drill 1.5011) (layers *.Cu *.Mask F.SilkS)
+      (net 37 "Net-(D21-Pad2)"))
+    (pad 2 thru_hole circle (at -3.81 -2.54 180) (size 2.6 2.6) (drill 1.5011) (layers *.Cu *.Mask F.SilkS)
+      (net 17 /ROW2))
+    (pad "" thru_hole circle (at -5.08 0 180) (size 1.69926 1.69926) (drill 1.69926) (layers *.Cu *.Mask F.SilkS))
+    (pad "" thru_hole circle (at 5.08 0 180) (size 1.69926 1.69926) (drill 1.69926) (layers *.Cu *.Mask F.SilkS))
+    (pad 1 thru_hole circle (at 2.5 -4.5 180) (size 2.5 2.5) (drill 1.5) (layers *.Cu *.Mask F.SilkS)
+      (net 37 "Net-(D21-Pad2)"))
+    (pad 2 thru_hole circle (at -2.5 -4 180) (size 2.5 2.5) (drill 1.5) (layers *.Cu *.Mask F.SilkS)
+      (net 17 /ROW2))
+    (model cherry_mx1.wrl
+      (at (xyz 0 0 0))
+      (scale (xyz 1 1 1))
+      (rotate (xyz 0 0 0))
+    )
+  )
   (gr_line (start 120.857 138.196) (end 121.657 137.396) (angle 90) (layer B.SilkS) (width 0.2))
   (gr_line (start 124.457 148.096) (end 124.457 148.296) (angle 90) (layer B.SilkS) (width 0.2))
@@
   (segment (start 232.757 96.471784) (end 222.4278 106.800984) (width 0.4064) (layer B.Cu) (net 16))
   (segment (start 223.057 86.496) (end 223.057 72.796) (width 0.4064) (layer B.Cu) (net 16))
+  (segment (start 137.7 86.7) (end 137.7 86.55) (width 0.4064) (layer F.Cu) (net 17))
+  (segment (start 137.7 86.55) (end 139.01 85.24) (width 0.4064) (layer F.Cu) (net 17))
   (segment (start 227.66 87.78) (end 242.783 87.78) (width 0.4064) (layer F.Cu) (net 17))
   (segment (start 248.05 90.2) (end 253.01 85.24) (width 0.4064) (layer F.Cu) (net 17))
@@
   (segment (start 223.2279 106.862992) (end 223.2279 112.237) (width 0.4064) (layer B.Cu) (net 17))
   (segment (start 227.66 87.78) (end 230.641 87.78) (width 0.4064) (layer B.Cu) (net 17))
-  (segment (start 144.060003 104.24) (end 144.060003 94.860003) (width 0.4064) (layer F.Cu) (net 18))
-  (segment (start 144.060003 94.860003) (end 134.8 85.6) (width 0.4064) (layer F.Cu) (net 18))
-  (segment (start 134.8 85.6) (end 131.7 85.6) (width 0.4064) (layer F.Cu) (net 18))
-  (segment (start 131.7 85.6) (end 128.220001 89.079999) (width 0.4064) (layer F.Cu) (net 18))
-  (segment (start 128.220001 89.079999) (end 114.959999 89.079999) (width 0.4064) (layer F.Cu) (net 18))
-  (segment (start 114.959999 89.079999) (end 113.66 87.78) (width 0.4064) (layer F.Cu) (net 18))
+  (segment (start 113.66 87.78) (end 114.959999 89.079999) (width 0.4064) (layer F.Cu) (net 18))
+  (segment (start 114.959999 89.079999) (end 128.220001 89.079999) (width 0.4064) (layer F.Cu) (net 18))
+  (segment (start 128.220001 89.079999) (end 132.010401 85.289599) (width 0.4064) (layer F.Cu) (net 18))
+  (segment (start 132.010401 85.289599) (end 133.584125 85.289599) (width 0.4064) (layer F.Cu) (net 18))
+  (segment (start 133.584125 85.289599) (end 140.496526 92.202) (width 0.4064) (layer F.Cu) (net 18))
+  (segment (start 141.732 92.202) (end 144.060003 94.530003) (width 0.4064) (layer F.Cu) (net 18))
+  (segment (start 140.496526 92.202) (end 141.732 92.202) (width 0.4064) (layer F.Cu) (net 18))
+  (segment (start 144.060003 94.530003) (end 144.060003 94.860003) (width 0.4064) (layer F.Cu) (net 18))
+  (segment (start 144.060003 94.860003) (end 144.060003 104.24) (width 0.4064) (layer F.Cu) (net 18))
   (segment (start 214.07 106.78) (end 236.183 106.78) (width 0.4064) (layer F.Cu) (net 18))
   (segment (start 241.1 109.4) (end 246.26 104.24) (width 0.4064) (layer F.Cu) (net 18))
@@
   (segment (start 120.0293 85.2593) (end 120.01 85.24) (width 0.4064) (layer B.Cu) (net 44))
   (segment (start 120.0293 85.2593) (end 120.01 85.24) (width 0.4064) (layer B.Cu) (net 44))
-  (segment (start 142.657 90.896) (end 138.757 90.896) (width 0.4064) (layer B.Cu) (net 44))
+  (segment (start 142.657 90.896) (end 139.265 90.896) (width 0.4064) (layer B.Cu) (net 44))
   (segment (start 150.203302 93.486398) (end 144.247398 93.486398) (width 0.4064) (layer B.Cu) (net 44))
   (segment (start 144.247398 93.486398) (end 143.457 92.696) (width 0.4064) (layer B.Cu) (net 44))
@@
   (segment (start 143.457 91.696) (end 142.657 90.896) (width 0.4064) (layer B.Cu) (net 44))
   (segment (start 150.203302 93.486398) (end 151.4937 92.196) (width 0.4064) (layer B.Cu) (net 44))
-  (segment (start 138.757 90.896) (end 133.1203 85.2593) (width 0.4064) (layer B.Cu) (net 44))
-  (segment (start 120.0293 85.2593) (end 133.1203 85.2593) (width 0.4064) (layer B.Cu) (net 44))
+  (segment (start 139.265 90.896) (end 133.6283 85.2593) (width 0.4064) (layer B.Cu) (net 44))
+  (segment (start 120.0293 85.2593) (end 133.6283 85.2593) (width 0.4064) (layer B.Cu) (net 44))
   (segment (start 142.0225 106.78) (end 137.710003 106.78) (width 0.4064) (layer B.Cu) (net 45))
   (segment (start 146.3929 111.1504) (end 142.0225 106.78) (width 0.4064) (layer B.Cu) (net 45))

Commit message: switch 22
Parts:
- SW22: footprint UGL:Cherry_MX -> ugl:Cherry-MX-Matias-Hybrid
Routing:
- net Net-(D22-Pad2): track 18.4 -> 20.4 mm
- net /ROW2: track 160.6 -> 161.4 mm
- net /COL1: track 193.0 -> 193.7 mm

Commit message: switch 23
Parts:
- SW23: footprint UGL:Cherry_MX -> ugl:Cherry-MX-Matias-Hybrid
Routing:
- net Net-(D23-Pad2): track 8.61 -> 10.6 mm
- net /COL3: track 210.9 -> 211.9 mm
- net /ROW2: track 161.4 -> 162.1 mm

Commit message: switch 24
Parts:
- SW24: footprint UGL:Cherry_MX -> ugl:Cherry-MX-Matias-Hybrid
Routing:
- net Net-(D24-Pad2): track 8.79 -> 10.8 mm
- net /COL4: track 146.5 -> 148.0 mm
- net /ROW2: track 162.1 -> 163.2 mm
Changed lines of the file:
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@@
 (kicad_pcb (version 4) (host pcbnew 4.0.1-stable)
   (general
-    (links 329)
+    (links 331)
     (no_connects 0)
     (area 19.803 18.9051 270.000001 165.000001)
     (thickness 1.6)
     (drawings 354)
-    (tracks 975)
+    (tracks 983)
     (zones 0)
     (modules 208)
@@
   )
   (layers
-    (0 F.Cu signal hide)
-    (31 B.Cu signal)
+    (0 F.Cu signal)
+    (31 B.Cu signal hide)
     (32 B.Adhes user)
     (33 F.Adhes user)
@@
       (net 17 /ROW2))
   )
-  (module UGL:Cherry_MX locked (layer F.Cu)
-    (at 192.2 82.7 180)
-    (fp_text reference SW24 (at 0 4.9 180) (layer F.SilkS)
-      (effects (font (size 1.5 1.5) (thickness 0.3)))
-    )
-    (fp_text value SPST (at 0 0 180) (layer F.SilkS) hide
-      (effects (font (size 1.5 1.5) (thickness 0.3)))
-    )
-    (fp_line (start -7.6 -7.6) (end -7.6 7.6) (layer B.SilkS) (width 0.15))
-    (fp_line (start -7.6 7.6) (end 7.6 7.6) (layer B.SilkS) (width 0.15))
-    (fp_line (start 7.6 -7.6) (end 7.6 7.6) (layer B.SilkS) (width 0.15))
-    (fp_line (start -7.6 -7.6) (end 7.6 -7.6) (layer B.SilkS) (width 0.15))
-    (fp_line (start -7.62 -7.62) (end 7.62 -7.62) (layer F.SilkS) (width 0.15))
-    (fp_line (start 7.62 -7.62) (end 7.62 7.62) (layer F.SilkS) (width 0.15))
-    (fp_line (start 7.62 7.62) (end -7.62 7.62) (layer F.SilkS) (width 0.15))
-    (fp_line (start -7.62 7.62) (end -7.62 -7.62) (layer F.SilkS) (width 0.15))
-    (pad "" np_thru_hole circle (at 0 0 180) (size 4 4) (drill 4) (layers *.Cu *.Mask F.SilkS))
-    (pad 2 thru_hole circle (at -3.81 -2.54 180) (size 2.5 2.5) (drill 1.5) (layers *.Cu *.Mask F.SilkS)
-      (net 40 "Net-(D24-Pad2)"))
-    (pad 1 thru_hole circle (at 2.54 -5.08 180) (size 2.5 2.5) (drill 1.5) (layers *.Cu *.Mask F.SilkS)
-      (net 17 /ROW2))
-  )
   (module UGL:UX60-MB-5S8 locked (layer F.Cu)
     (at 175.849803 43.601924 85.4)
@@
     )
   )
+  (module ugl:Cherry-MX-Matias-Hybrid locked (layer F.Cu)
+    (at 192.2 82.7 180)
+    (tags switch)
+    (fp_text reference SW24 (at 0 3.81 180) (layer F.SilkS)
+      (effects (font (thickness 0.3048)))
+    )
+    (fp_text value SPST (at 0 0 180) (layer F.SilkS) hide
+      (effects (font (thickness 0.3048)))
+    )
+    (fp_line (start -7.62 7.62) (end -7.62 -7.62) (layer B.SilkS) (width 0.15))
+    (fp_line (start 7.62 7.62) (end -7.62 7.62) (layer B.SilkS) (width 0.15))
+    (fp_line (start 7.62 -7.62) (end 7.62 7.62) (layer B.SilkS) (width 0.15))
+    (fp_line (start -7.62 -7.62) (end 7.62 -7.62) (layer B.SilkS) (width 0.15))
+    (fp_line (start -7.75 -6.4) (end -7.75 6.4) (layer F.SilkS) (width 0.15))
+    (fp_line (start 7.75 -6.4) (end 7.75 6.4) (layer F.SilkS) (width 0.15))
+    (fp_line (start -7.75 6.4) (end 7.75 6.4) (layer F.SilkS) (width 0.15))
+    (fp_line (start -7.75 -6.4) (end 7.75 -6.4) (layer F.SilkS) (width 0.15))
+    (fp_line (start -7.62 -7.62) (end 7.62 -7.62) (layer F.SilkS) (width 0.15))
+    (fp_line (start 7.62 -7.62) (end 7.62 7.62) (layer F.SilkS) (width 0.15))
+    (fp_line (start 7.62 7.62) (end -7.62 7.62) (layer F.SilkS) (width 0.15))
+    (fp_line (start -7.62 7.62) (end -7.62 -7.62) (layer F.SilkS) (width 0.15))
+    (pad 0 thru_hole circle (at 0 0 180) (size 3.98018 3.98018) (drill 3.98018) (layers *.Cu *.Mask F.SilkS))
+    (pad 1 thru_hole circle (at 2.54 -5.08 180) (size 2.6 2.6) (drill 1.5011) (layers *.Cu *.Mask F.SilkS)
+      (net 17 /ROW2))
+    (pad 2 thru_hole circle (at -3.81 -2.54 180) (size 2.6 2.6) (drill 1.5011) (layers *.Cu *.Mask F.SilkS)
+      (net 40 "Net-(D24-Pad2)"))
+    (pad "" thru_hole circle (at -5.08 0 180) (size 1.69926 1.69926) (drill 1.69926) (layers *.Cu *.Mask F.SilkS))
+    (pad "" thru_hole circle (at 5.08 0 180) (size 1.69926 1.69926) (drill 1.69926) (layers *.Cu *.Mask F.SilkS))
+    (pad 1 thru_hole circle (at 2.5 -4.5 180) (size 2.5 2.5) (drill 1.5) (layers *.Cu *.Mask F.SilkS)
+      (net 17 /ROW2))
+    (pad 2 thru_hole circle (at -2.5 -4 180) (size 2.5 2.5) (drill 1.5) (layers *.Cu *.Mask F.SilkS)
+      (net 40 "Net-(D24-Pad2)"))
+    (model cherry_mx1.wrl
+      (at (xyz 0 0 0))
+      (scale (xyz 1 1 1))
+      (rotate (xyz 0 0 0))
+    )
+  )
   (gr_line (start 120.857 138.196) (end 121.657 137.396) (angle 90) (layer B.SilkS) (width 0.2))
   (gr_line (start 124.457 148.096) (end 124.457 148.296) (angle 90) (layer B.SilkS) (width 0.2))
@@
   (segment (start 164.1203 120.6327) (end 164.1203 130.196) (width 0.4064) (layer B.Cu) (net 3))
   (segment (start 174.3203 111.196) (end 173.557 111.196) (width 0.4064) (layer B.Cu) (net 3))
+  (segment (start 198.536031 87.764269) (end 198.536031 82.097104) (width 0.4064) (layer B.Cu) (net 4))
+  (segment (start 183.8203 73.196) (end 187.257 73.196) (width 0.4064) (layer B.Cu) (net 4))
+  (segment (start 195.1203 91.18) (end 198.536031 87.764269) (width 0.4064) (layer B.Cu) (net 4))
+  (segment (start 198.536031 82.097104) (end 189.634927 73.196) (width 0.4064) (layer B.Cu) (net 4))
+  (segment (start 195.1203 92.196) (end 195.1203 91.18) (width 0.4064) (layer B.Cu) (net 4))
+  (segment (start 189.634927 73.196) (end 187.257 73.196) (width 0.4064) (layer B.Cu) (net 4))
   (segment (start 215.2659 119.0371) (end 215.028008 119.0371) (width 0.4064) (layer B.Cu) (net 4))
   (segment (start 192.014 136.896) (end 174.8001 136.896) (width 0.4064) (layer B.Cu) (net 4))
@@
   (segment (start 172.72 133.6963) (end 172.72 138.8511) (width 0.4064) (layer B.Cu) (net 4))
   (segment (start 176.2203 130.196) (end 172.72 133.6963) (width 0.4064) (layer B.Cu) (net 4))
-  (segment (start 198.357 84.296) (end 198.357 88.9593) (width 0.4064) (layer B.Cu) (net 4))
-  (segment (start 198.357 88.9593) (end 195.1203 92.196) (width 0.4064) (layer B.Cu) (net 4))
-  (segment (start 183.8203 73.196) (end 187.257 73.196) (width 0.4064) (layer B.Cu) (net 4))
-  (segment (start 187.257 73.196) (end 198.357 84.296) (width 0.4064) (layer B.Cu) (net 4))
   (segment (start 186.6203 100.696) (end 186.6203 111.196) (width 0.4064) (layer B.Cu) (net 4))
   (segment (start 195.1203 92.196) (end 186.6203 100.696) (width 0.4064) (layer B.Cu) (net 4))
   (segment (start 176.2203 121.596) (end 176.2203 130.196) (width 0.4064) (layer B.Cu) (net 4))
   (segment (start 186.6203 111.196) (end 176.2203 121.596) (width 0.4064) (layer B.Cu) (net 4))
+  (segment (start 208.9937 92.1686) (end 208.9937 92.196) (width 0.4064) (layer B.Cu) (net 5))
+  (segment (start 195.4937 78.192653) (end 199.145642 81.844595) (width 0.4064) (layer B.Cu) (net 5))
+  (segment (start 195.4937 73.096) (end 195.4937 78.192653) (width 0.4064) (layer B.Cu) (net 5))
+  (segment (start 199.145642 82.320542) (end 208.9937 92.1686) (width 0.4064) (layer B.Cu) (net 5))
+  (segment (start 199.145642 81.844595) (end 199.145642 82.320542) (width 0.4064) (layer B.Cu) (net 5))
   (segment (start 218.028 118.237) (end 214.966 118.237) (width 0.4064) (layer B.Cu) (net 5))
   (segment (start 214.966 118.237) (end 211.857 121.346) (width 0.4064) (layer B.Cu) (net 5))
@@
   (segment (start 197.4088 140.1445) (end 196.2404 138.9761) (width 0.4064) (layer B.Cu) (net 5))
   (segment (start 196.088 130.196) (end 196.088 138.8511) (width 0.4064) (layer B.Cu) (net 5))
-  (segment (start 195.4937 73.096) (end 195.4937 78.696) (width 0.4064) (layer B.Cu) (net 5))
-  (segment (start 195.4937 78.696) (end 202.6559 85.8582) (width 0.4064) (layer B.Cu) (net 5))
-  (segment (start 208.9937 92.196) (end 202.6559 85.8582) (width 0.4064) (layer B.Cu) (net 5))
   (segment (start 188.2203 130.196) (end 196.088 130.196) (width 0.4064) (layer B.Cu) (net 5))
   (segment (start 203.8203 92.196) (end 208.9937 92.196) (width 0.4064) (layer B.Cu) (net 5))
@@
   (segment (start 232.757 96.471784) (end 222.4278 106.800984) (width 0.4064) (layer B.Cu) (net 16))
   (segment (start 223.057 86.496) (end 223.057 72.796) (width 0.4064) (layer B.Cu) (net 16))
+  (segment (start 208.66 87.78) (end 207.360001 89.079999) (width 0.4064) (layer F.Cu) (net 17))
+  (segment (start 207.360001 89.079999) (end 190.959999 89.079999) (width 0.4064) (layer F.Cu) (net 17))
+  (segment (start 190.959999 89.079999) (end 189.66 87.78) (width 0.4064) (layer F.Cu) (net 17))
   (segment (start 170.7 87.2) (end 171.949999 88.449999) (width 0.4064) (layer F.Cu) (net 17))
   (segment (start 187.222235 88.449999) (end 187.892234 87.78) (width 0.4064) (layer F.Cu) (net 17))
@@
   (segment (start 254.003 86.233) (end 254.003 92.2) (width 0.4064) (layer B.Cu) (net 17))
   (segment (start 227.66 87.78) (end 208.66 87.78) (width 0.4064) (layer F.Cu) (net 17))
-  (segment (start 208.66 87.78) (end 189.66 87.78) (width 0.4064) (layer F.Cu) (net 17))
   (segment (start 141.55 87.78) (end 139.01 85.24) (width 0.4064) (layer F.Cu) (net 17))
   (segment (start 151.66 87.78) (end 141.55 87.78) (width 0.4064) (layer F.Cu) (net 17))
@@
   (segment (start 177.01 88.2123) (end 180.9937 92.196) (width 0.4064) (layer B.Cu) (net 39))
   (segment (start 177.01 85.24) (end 177.01 88.2123) (width 0.4064) (layer B.Cu) (net 39))
-  (segment (start 196.01 87.7797) (end 196.01 85.24) (width 0.4064) (layer B.Cu) (net 40))
+  (segment (start 194.7 86.7) (end 194.7 86.55) (width 0.4064) (layer B.Cu) (net 40))
+  (segment (start 194.7 86.55) (end 196.01 85.24) (width 0.4064) (layer B.Cu) (net 40))
   (segment (start 191.5937 92.196) (end 196.01 87.7797) (width 0.4064) (layer B.Cu) (net 40))
+  (segment (start 196.01 87.7797) (end 196.01 85.24) (width 0.4064) (layer B.Cu) (net 40))
   (segment (start 215.01 90.1075) (end 215.01 85.24) (width 0.4064) (layer B.Cu) (net 41))
   (segment (start 212.9663 92.1512) (end 215.01 90.1075) (width 0.4064) (layer B.Cu) (net 41))
