File: right-main/right-main.kicad_pcb (KiCad board)
At the start: 2 copper layers, 150.4 x 123.8 mm, 208 parts, among them J1 USBCONN, P1 CONN_4, P2 CONN_5, P3 CONN_6, SW1 PTS525SM10, SW11 SPST, SW12 SPST, SW13 SPST, SW14 SPST, SW15 SPST, SW16 SPST, SW17 SPST, SW21 SPST, SW22 SPST, SW23 SPST, SW24 SPST, SW25 SPST, SW26 SPST, SW27 SPST, SW31 SPST, SW32 SPST, SW33 SPST, SW34 SPST, SW35 SPST, SW36 SPST, SW37 SPST, SW41 SPST, SW42 SPST, SW43 SPST, SW44 SPST, SW45 SPST, SW46 SPST, SW47 SPST, SW52 SPST, SW53 SPST, SW54 SPST, SW55 SPST, SW56 SPST, SW57 SPST, U1 ATMEGA32U4, U2 CAT24C256, X1 16Mhz

Commit message: switch 25
Parts:
- SW25: footprint UGL:Cherry_MX -> ugl:Cherry-MX-Matias-Hybrid
Routing:
- net Net-(D25-Pad2): track 7.76 -> 9.76 mm
- net /ROW2: track 163.2 -> 164.3 mm
Changed lines of the file:
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@@
 (kicad_pcb (version 4) (host pcbnew 4.0.1-stable)
   (general
-    (links 331)
+    (links 333)
     (no_connects 0)
     (area 19.803 18.9051 270.000001 165.000001)
     (thickness 1.6)
     (drawings 354)
-    (tracks 983)
+    (tracks 988)
     (zones 0)
     (modules 208)
@@
   (layers
     (0 F.Cu signal)
-    (31 B.Cu signal hide)
+    (31 B.Cu signal)
     (32 B.Adhes user)
     (33 F.Adhes user)
     (34 B.Paste user)
     (35 F.Paste user)
-    (36 B.SilkS user hide)
-    (37 F.SilkS user hide)
+    (36 B.SilkS user)
+    (37 F.SilkS user)
     (38 B.Mask user)
     (39 F.Mask user)
@@
       (net 17 /ROW2))
   )
-  (module UGL:Cherry_MX locked (layer F.Cu)
-    (at 211.2 82.7 180)
-    (fp_text reference SW25 (at 0 4.9 180) (layer F.SilkS)
-      (effects (font (size 1.5 1.5) (thickness 0.3)))
-    )
-    (fp_text value SPST (at 0 0 180) (layer F.SilkS) hide
-      (effects (font (size 1.5 1.5) (thickness 0.3)))
-    )
-    (fp_line (start -7.6 -7.6) (end -7.6 7.6) (layer B.SilkS) (width 0.15))
-    (fp_line (start -7.6 7.6) (end 7.6 7.6) (layer B.SilkS) (width 0.15))
-    (fp_line (start 7.6 -7.6) (end 7.6 7.6) (layer B.SilkS) (width 0.15))
-    (fp_line (start -7.6 -7.6) (end 7.6 -7.6) (layer B.SilkS) (width 0.15))
-    (fp_line (start -7.62 -7.62) (end 7.62 -7.62) (layer F.SilkS) (width 0.15))
-    (fp_line (start 7.62 -7.62) (end 7.62 7.62) (layer F.SilkS) (width 0.15))
-    (fp_line (start 7.62 7.62) (end -7.62 7.62) (layer F.SilkS) (width 0.15))
-    (fp_line (start -7.62 7.62) (end -7.62 -7.62) (layer F.SilkS) (width 0.15))
-    (pad "" np_thru_hole circle (at 0 0 180) (size 4 4) (drill 4) (layers *.Cu *.Mask F.SilkS))
-    (pad 2 thru_hole circle (at -3.81 -2.54 180) (size 2.5 2.5) (drill 1.5) (layers *.Cu *.Mask F.SilkS)
-      (net 41 "Net-(D25-Pad2)"))
-    (pad 1 thru_hole circle (at 2.54 -5.08 180) (size 2.5 2.5) (drill 1.5) (layers *.Cu *.Mask F.SilkS)
-      (net 17 /ROW2))
-  )
   (module UGL:UX60-MB-5S8 locked (layer F.Cu)
     (at 175.849803 43.601924 85.4)
@@
     )
   )
+  (module ugl:Cherry-MX-Matias-Hybrid locked (layer F.Cu)
+    (at 211.2 82.7 180)
+    (tags switch)
+    (fp_text reference SW25 (at 0 3.81 180) (layer F.SilkS)
+      (effects (font (thickness 0.3048)))
+    )
+    (fp_text value SPST (at 0 0 180) (layer F.SilkS) hide
+      (effects (font (thickness 0.3048)))
+    )
+    (fp_line (start -7.62 7.62) (end -7.62 -7.62) (layer B.SilkS) (width 0.15))
+    (fp_line (start 7.62 7.62) (end -7.62 7.62) (layer B.SilkS) (width 0.15))
+    (fp_line (start 7.62 -7.62) (end 7.62 7.62) (layer B.SilkS) (width 0.15))
+    (fp_line (start -7.62 -7.62) (end 7.62 -7.62) (layer B.SilkS) (width 0.15))
+    (fp_line (start -7.75 -6.4) (end -7.75 6.4) (layer F.SilkS) (width 0.15))
+    (fp_line (start 7.75 -6.4) (end 7.75 6.4) (layer F.SilkS) (width 0.15))
+    (fp_line (start -7.75 6.4) (end 7.75 6.4) (layer F.SilkS) (width 0.15))
+    (fp_line (start -7.75 -6.4) (end 7.75 -6.4) (layer F.SilkS) (width 0.15))
+    (fp_line (start -7.62 -7.62) (end 7.62 -7.62) (layer F.SilkS) (width 0.15))
+    (fp_line (start 7.62 -7.62) (end 7.62 7.62) (layer F.SilkS) (width 0.15))
+    (fp_line (start 7.62 7.62) (end -7.62 7.62) (layer F.SilkS) (width 0.15))
+    (fp_line (start -7.62 7.62) (end -7.62 -7.62) (layer F.SilkS) (width 0.15))
+    (pad 0 thru_hole circle (at 0 0 180) (size 3.98018 3.98018) (drill 3.98018) (layers *.Cu *.Mask F.SilkS))
+    (pad 1 thru_hole circle (at 2.54 -5.08 180) (size 2.6 2.6) (drill 1.5011) (layers *.Cu *.Mask F.SilkS)
+      (net 17 /ROW2))
+    (pad 2 thru_hole circle (at -3.81 -2.54 180) (size 2.6 2.6) (drill 1.5011) (layers *.Cu *.Mask F.SilkS)
+      (net 41 "Net-(D25-Pad2)"))
+    (pad "" thru_hole circle (at -5.08 0 180) (size 1.69926 1.69926) (drill 1.69926) (layers *.Cu *.Mask F.SilkS))
+    (pad "" thru_hole circle (at 5.08 0 180) (size 1.69926 1.69926) (drill 1.69926) (layers *.Cu *.Mask F.SilkS))
+    (pad 1 thru_hole circle (at 2.5 -4.5 180) (size 2.5 2.5) (drill 1.5) (layers *.Cu *.Mask F.SilkS)
+      (net 17 /ROW2))
+    (pad 2 thru_hole circle (at -2.5 -4 180) (size 2.5 2.5) (drill 1.5) (layers *.Cu *.Mask F.SilkS)
+      (net 41 "Net-(D25-Pad2)"))
+    (model cherry_mx1.wrl
+      (at (xyz 0 0 0))
+      (scale (xyz 1 1 1))
+      (rotate (xyz 0 0 0))
+    )
+  )
   (gr_line (start 120.857 138.196) (end 121.657 137.396) (angle 90) (layer B.SilkS) (width 0.2))
   (gr_line (start 124.457 148.096) (end 124.457 148.296) (angle 90) (layer B.SilkS) (width 0.2))
@@
   (segment (start 232.757 96.471784) (end 222.4278 106.800984) (width 0.4064) (layer B.Cu) (net 16))
   (segment (start 223.057 86.496) (end 223.057 72.796) (width 0.4064) (layer B.Cu) (net 16))
+  (segment (start 227.66 87.78) (end 225.892234 87.78) (width 0.4064) (layer F.Cu) (net 17))
+  (segment (start 225.892234 87.78) (end 224.592235 89.079999) (width 0.4064) (layer F.Cu) (net 17))
+  (segment (start 224.592235 89.079999) (end 209.959999 89.079999) (width 0.4064) (layer F.Cu) (net 17))
+  (segment (start 209.959999 89.079999) (end 208.66 87.78) (width 0.4064) (layer F.Cu) (net 17))
   (segment (start 208.66 87.78) (end 207.360001 89.079999) (width 0.4064) (layer F.Cu) (net 17))
   (segment (start 207.360001 89.079999) (end 190.959999 89.079999) (width 0.4064) (layer F.Cu) (net 17))
@@
   (segment (start 253.01 85.24) (end 254.003 86.233) (width 0.4064) (layer B.Cu) (net 17))
   (segment (start 254.003 86.233) (end 254.003 92.2) (width 0.4064) (layer B.Cu) (net 17))
-  (segment (start 227.66 87.78) (end 208.66 87.78) (width 0.4064) (layer F.Cu) (net 17))
   (segment (start 141.55 87.78) (end 139.01 85.24) (width 0.4064) (layer F.Cu) (net 17))
   (segment (start 151.66 87.78) (end 141.55 87.78) (width 0.4064) (layer F.Cu) (net 17))
@@
   (segment (start 191.5937 92.196) (end 196.01 87.7797) (width 0.4064) (layer B.Cu) (net 40))
   (segment (start 196.01 87.7797) (end 196.01 85.24) (width 0.4064) (layer B.Cu) (net 40))
+  (segment (start 213.7 86.7) (end 213.7 86.55) (width 0.4064) (layer B.Cu) (net 41))
+  (segment (start 213.7 86.55) (end 215.01 85.24) (width 0.4064) (layer B.Cu) (net 41))
   (segment (start 215.01 90.1075) (end 215.01 85.24) (width 0.4064) (layer B.Cu) (net 41))
   (segment (start 212.9663 92.1512) (end 215.01 90.1075) (width 0.4064) (layer B.Cu) (net 41))

Commit message: switch 26
Parts:
- SW26: footprint UGL:Cherry_MX -> ugl:Cherry-MX-Matias-Hybrid
Routing:
- net Net-(D26-Pad2): track 7.33 -> 9.34 mm
- net /COL3: track 211.9 -> 213.3 mm
- net /D-: track 131.2 -> 132.5 mm
- net /RX: track 314.4 -> 315.7 mm
- net /COL2: track 252.3 -> 253.7 mm
- net /D+: track 134.0 -> 135.3 mm
- net /TX: track 316.9 -> 318.3 mm
- net VCC: track 433.9 -> 435.2 mm
- net /COL1: track 193.7 -> 195.0 mm
- net /ROW2: track 164.3 -> 165.4 mm
- net /COL7: track 87.6 -> 88.2 mm

Commit message: switch 27
Parts:
- SW27: footprint UGL:Cherry_MX -> ugl:Cherry-MX-Matias-Hybrid
Routing:
- net /ROW2: track 165.4 -> 167.4 mm
Changed lines of the file:
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@@
 (kicad_pcb (version 4) (host pcbnew 4.0.1-stable)
   (general
-    (links 335)
+    (links 337)
     (no_connects 0)
     (area 19.803 18.9051 270.000001 165.000001)
     (thickness 1.6)
     (drawings 354)
-    (tracks 1018)
+    (tracks 1020)
     (zones 0)
     (modules 208)
@@
   )
   (layers
-    (0 F.Cu signal hide)
-    (31 B.Cu signal)
+    (0 F.Cu signal)
+    (31 B.Cu signal hide)
     (32 B.Adhes user)
     (33 F.Adhes user)
@@
       (net 45 "Net-(D32-Pad2)"))
   )
-  (module UGL:Cherry_MX locked (layer F.Cu)
-    (at 249.2 82.7 180)
-    (fp_text reference SW27 (at 0 4.9 180) (layer F.SilkS)
-      (effects (font (size 1.5 1.5) (thickness 0.3)))
-    )
-    (fp_text value SPST (at 0 0 180) (layer F.SilkS) hide
-      (effects (font (size 1.5 1.5) (thickness 0.3)))
-    )
-    (fp_line (start -7.6 -7.6) (end -7.6 7.6) (layer B.SilkS) (width 0.15))
-    (fp_line (start -7.6 7.6) (end 7.6 7.6) (layer B.SilkS) (width 0.15))
-    (fp_line (start 7.6 -7.6) (end 7.6 7.6) (layer B.SilkS) (width 0.15))
-    (fp_line (start -7.6 -7.6) (end 7.6 -7.6) (layer B.SilkS) (width 0.15))
-    (fp_line (start -7.62 -7.62) (end 7.62 -7.62) (layer F.SilkS) (width 0.15))
-    (fp_line (start 7.62 -7.62) (end 7.62 7.62) (layer F.SilkS) (width 0.15))
-    (fp_line (start 7.62 7.62) (end -7.62 7.62) (layer F.SilkS) (width 0.15))
-    (fp_line (start -7.62 7.62) (end -7.62 -7.62) (layer F.SilkS) (width 0.15))
-    (pad "" np_thru_hole circle (at 0 0 180) (size 4 4) (drill 4) (layers *.Cu *.Mask F.SilkS))
-    (pad 2 thru_hole circle (at -3.81 -2.54 180) (size 2.5 2.5) (drill 1.5) (layers *.Cu *.Mask F.SilkS)
-      (net 17 /ROW2))
-    (pad 1 thru_hole circle (at 2.54 -5.08 180) (size 2.5 2.5) (drill 1.5) (layers *.Cu *.Mask F.SilkS)
-      (net 43 "Net-(D27-Pad2)"))
-  )
   (module UGL:UX60-MB-5S8 locked (layer F.Cu)
     (at 175.849803 43.601924 85.4)
@@
     )
   )
+  (module ugl:Cherry-MX-Matias-Hybrid locked (layer F.Cu)
+    (at 249.2 82.7 180)
+    (tags switch)
+    (fp_text reference SW27 (at 0 3.81 180) (layer F.SilkS)
+      (effects (font (thickness 0.3048)))
+    )
+    (fp_text value SPST (at 0 0 180) (layer F.SilkS) hide
+      (effects (font (thickness 0.3048)))
+    )
+    (fp_line (start -7.62 7.62) (end -7.62 -7.62) (layer B.SilkS) (width 0.15))
+    (fp_line (start 7.62 7.62) (end -7.62 7.62) (layer B.SilkS) (width 0.15))
+    (fp_line (start 7.62 -7.62) (end 7.62 7.62) (layer B.SilkS) (width 0.15))
+    (fp_line (start -7.62 -7.62) (end 7.62 -7.62) (layer B.SilkS) (width 0.15))
+    (fp_line (start -7.75 -6.4) (end -7.75 6.4) (layer F.SilkS) (width 0.15))
+    (fp_line (start 7.75 -6.4) (end 7.75 6.4) (layer F.SilkS) (width 0.15))
+    (fp_line (start -7.75 6.4) (end 7.75 6.4) (layer F.SilkS) (width 0.15))
+    (fp_line (start -7.75 -6.4) (end 7.75 -6.4) (layer F.SilkS) (width 0.15))
+    (fp_line (start -7.62 -7.62) (end 7.62 -7.62) (layer F.SilkS) (width 0.15))
+    (fp_line (start 7.62 -7.62) (end 7.62 7.62) (layer F.SilkS) (width 0.15))
+    (fp_line (start 7.62 7.62) (end -7.62 7.62) (layer F.SilkS) (width 0.15))
+    (fp_line (start -7.62 7.62) (end -7.62 -7.62) (layer F.SilkS) (width 0.15))
+    (pad 0 thru_hole circle (at 0 0 180) (size 3.98018 3.98018) (drill 3.98018) (layers *.Cu *.Mask F.SilkS))
+    (pad 1 thru_hole circle (at 2.54 -5.08 180) (size 2.6 2.6) (drill 1.5011) (layers *.Cu *.Mask F.SilkS)
+      (net 43 "Net-(D27-Pad2)"))
+    (pad 2 thru_hole circle (at -3.81 -2.54 180) (size 2.6 2.6) (drill 1.5011) (layers *.Cu *.Mask F.SilkS)
+      (net 17 /ROW2))
+    (pad "" thru_hole circle (at -5.08 0 180) (size 1.69926 1.69926) (drill 1.69926) (layers *.Cu *.Mask F.SilkS))
+    (pad "" thru_hole circle (at 5.08 0 180) (size 1.69926 1.69926) (drill 1.69926) (layers *.Cu *.Mask F.SilkS))
+    (pad 1 thru_hole circle (at 2.5 -4.5 180) (size 2.5 2.5) (drill 1.5) (layers *.Cu *.Mask F.SilkS)
+      (net 43 "Net-(D27-Pad2)"))
+    (pad 2 thru_hole circle (at -2.5 -4 180) (size 2.5 2.5) (drill 1.5) (layers *.Cu *.Mask F.SilkS)
+      (net 17 /ROW2))
+    (model cherry_mx1.wrl
+      (at (xyz 0 0 0))
+      (scale (xyz 1 1 1))
+      (rotate (xyz 0 0 0))
+    )
+  )
   (gr_line (start 120.857 138.196) (end 121.657 137.396) (angle 90) (layer B.SilkS) (width 0.2))
   (gr_line (start 124.457 148.096) (end 124.457 148.296) (angle 90) (layer B.SilkS) (width 0.2))
@@
   (segment (start 232.757 96.471784) (end 222.4278 106.800984) (width 0.4064) (layer B.Cu) (net 16))
   (segment (start 223.057 86.496) (end 223.057 72.796) (width 0.4064) (layer B.Cu) (net 16))
+  (segment (start 251.7 86.7) (end 251.7 86.55) (width 0.4064) (layer B.Cu) (net 17))
+  (segment (start 251.7 86.55) (end 253.01 85.24) (width 0.4064) (layer B.Cu) (net 17))
   (segment (start 242.783 87.78) (end 241.483001 89.079999) (width 0.4064) (layer F.Cu) (net 17))
   (segment (start 241.483001 89.079999) (end 228.959999 89.079999) (width 0.4064) (layer F.Cu) (net 17))

Commit message: switch 41
Parts:
- SW41: footprint UGL:Cherry_MX -> ugl:Cherry-MX-Matias-Hybrid
Routing:
- net Net-(D41-Pad2): track 44.4 -> 46.4 mm
- net /ROW4: track 216.5 -> 217.6 mm
Changed lines of the file:
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@@
 (kicad_pcb (version 4) (host pcbnew 4.0.1-stable)
   (general
-    (links 337)
+    (links 339)
     (no_connects 0)
     (area 19.803 18.9051 270.000001 165.000001)
     (thickness 1.6)
     (drawings 354)
-    (tracks 1020)
+    (tracks 1025)
     (zones 0)
     (modules 208)
@@
   )
   (layers
-    (0 F.Cu signal)
-    (31 B.Cu signal hide)
+    (0 F.Cu signal hide)
+    (31 B.Cu signal)
     (32 B.Adhes user)
     (33 F.Adhes user)
@@
     (pad_to_mask_clearance 0)
     (aux_axis_origin 0 0)
-    (visible_elements FFFFEFFF)
+    (visible_elements FFFCEFFF)
     (pcbplotparams
       (layerselection 0x010f0_80000001)
@@
   )
   (module UGL:Cherry_MX locked (layer F.Cu)
-    (at 121.160007 101.7 180)
-    (fp_text reference SW41 (at 0 4.9 180) (layer F.SilkS)
-      (effects (font (size 1.5 1.5) (thickness 0.3)))
-    )
-    (fp_text value SPST (at 0 0 180) (layer F.SilkS) hide
-      (effects (font (size 1.5 1.5) (thickness 0.3)))
-    )
-    (fp_line (start -7.6 -7.6) (end -7.6 7.6) (layer B.SilkS) (width 0.15))
-    (fp_line (start -7.6 7.6) (end 7.6 7.6) (layer B.SilkS) (width 0.15))
-    (fp_line (start 7.6 -7.6) (end 7.6 7.6) (layer B.SilkS) (width 0.15))
-    (fp_line (start -7.6 -7.6) (end 7.6 -7.6) (layer B.SilkS) (width 0.15))
-    (fp_line (start -7.62 -7.62) (end 7.62 -7.62) (layer F.SilkS) (width 0.15))
-    (fp_line (start 7.62 -7.62) (end 7.62 7.62) (layer F.SilkS) (width 0.15))
-    (fp_line (start 7.62 7.62) (end -7.62 7.62) (layer F.SilkS) (width 0.15))
-    (fp_line (start -7.62 7.62) (end -7.62 -7.62) (layer F.SilkS) (width 0.15))
-    (pad "" np_thru_hole circle (at 0 0 180) (size 4 4) (drill 4) (layers *.Cu *.Mask F.SilkS))
-    (pad 2 thru_hole circle (at -3.81 -2.54 180) (size 2.5 2.5) (drill 1.5) (layers *.Cu *.Mask F.SilkS)
-      (net 51 "Net-(D41-Pad2)"))
-    (pad 1 thru_hole circle (at 2.54 -5.08 180) (size 2.5 2.5) (drill 1.5) (layers *.Cu *.Mask F.SilkS)
-      (net 19 /ROW4))
-  )
-  (module UGL:Cherry_MX locked (layer F.Cu)
     (at 242.45 101.7 180)
     (fp_text reference SW37 (at 0 4.9 180) (layer F.SilkS)
@@
     )
   )
+  (module ugl:Cherry-MX-Matias-Hybrid locked (layer F.Cu)
+    (at 121.160007 101.7 180)
+    (tags switch)
+    (fp_text reference SW41 (at 0 3.81 180) (layer F.SilkS)
+      (effects (font (thickness 0.3048)))
+    )
+    (fp_text value SPST (at 0 0 180) (layer F.SilkS) hide
+      (effects (font (thickness 0.3048)))
+    )
+    (fp_line (start -7.62 7.62) (end -7.62 -7.62) (layer B.SilkS) (width 0.15))
+    (fp_line (start 7.62 7.62) (end -7.62 7.62) (layer B.SilkS) (width 0.15))
+    (fp_line (start 7.62 -7.62) (end 7.62 7.62) (layer B.SilkS) (width 0.15))
+    (fp_line (start -7.62 -7.62) (end 7.62 -7.62) (layer B.SilkS) (width 0.15))
+    (fp_line (start -7.75 -6.4) (end -7.75 6.4) (layer F.SilkS) (width 0.15))
+    (fp_line (start 7.75 -6.4) (end 7.75 6.4) (layer F.SilkS) (width 0.15))
+    (fp_line (start -7.75 6.4) (end 7.75 6.4) (layer F.SilkS) (width 0.15))
+    (fp_line (start -7.75 -6.4) (end 7.75 -6.4) (layer F.SilkS) (width 0.15))
+    (fp_line (start -7.62 -7.62) (end 7.62 -7.62) (layer F.SilkS) (width 0.15))
+    (fp_line (start 7.62 -7.62) (end 7.62 7.62) (layer F.SilkS) (width 0.15))
+    (fp_line (start 7.62 7.62) (end -7.62 7.62) (layer F.SilkS) (width 0.15))
+    (fp_line (start -7.62 7.62) (end -7.62 -7.62) (layer F.SilkS) (width 0.15))
+    (pad 0 thru_hole circle (at 0 0 180) (size 3.98018 3.98018) (drill 3.98018) (layers *.Cu *.Mask F.SilkS))
+    (pad 1 thru_hole circle (at 2.54 -5.08 180) (size 2.6 2.6) (drill 1.5011) (layers *.Cu *.Mask F.SilkS)
+      (net 19 /ROW4))
+    (pad 2 thru_hole circle (at -3.81 -2.54 180) (size 2.6 2.6) (drill 1.5011) (layers *.Cu *.Mask F.SilkS)
+      (net 51 "Net-(D41-Pad2)"))
+    (pad "" thru_hole circle (at -5.08 0 180) (size 1.69926 1.69926) (drill 1.69926) (layers *.Cu *.Mask F.SilkS))
+    (pad "" thru_hole circle (at 5.08 0 180) (size 1.69926 1.69926) (drill 1.69926) (layers *.Cu *.Mask F.SilkS))
+    (pad 1 thru_hole circle (at 2.5 -4.5 180) (size 2.5 2.5) (drill 1.5) (layers *.Cu *.Mask F.SilkS)
+      (net 19 /ROW4))
+    (pad 2 thru_hole circle (at -2.5 -4 180) (size 2.5 2.5) (drill 1.5) (layers *.Cu *.Mask F.SilkS)
+      (net 51 "Net-(D41-Pad2)"))
+    (model cherry_mx1.wrl
+      (at (xyz 0 0 0))
+      (scale (xyz 1 1 1))
+      (rotate (xyz 0 0 0))
+    )
+  )
   (gr_line (start 120.857 138.196) (end 121.657 137.396) (angle 90) (layer B.SilkS) (width 0.2))
   (gr_line (start 124.457 148.096) (end 124.457 148.296) (angle 90) (layer B.SilkS) (width 0.2))
@@
   (segment (start 207.6977 115.8367) (end 218.028 115.8367) (width 0.4064) (layer B.Cu) (net 18))
   (segment (start 214.07 106.78) (end 209.997216 106.78) (width 0.4064) (layer B.Cu) (net 18))
+  (segment (start 145.5928 113.792) (end 145.5928 108.7928) (width 0.4064) (layer F.Cu) (net 19))
+  (segment (start 141.6 104.8) (end 136.4 104.8) (width 0.4064) (layer F.Cu) (net 19))
+  (segment (start 145.5928 108.7928) (end 141.6 104.8) (width 0.4064) (layer F.Cu) (net 19))
+  (segment (start 136.4 104.8) (end 133.120001 108.079999) (width 0.4064) (layer F.Cu) (net 19))
+  (segment (start 133.120001 108.079999) (end 119.920006 108.079999) (width 0.4064) (layer F.Cu) (net 19))
+  (segment (start 119.920006 108.079999) (end 118.620007 106.78) (width 0.4064) (layer F.Cu) (net 19))
   (segment (start 206.103 117.4369) (end 205.3161 117.4369) (width 0.4064) (layer B.Cu) (net 19))
   (segment (start 205.3161 117.4369) (end 203.357 119.396) (width 0.4064) (layer B.Cu) (net 19))
@@
   (segment (start 147.359997 125.78) (end 128.16 125.78) (width 0.4064) (layer F.Cu) (net 19))
   (segment (start 145.5928 113.792) (end 145.5928 113.6904) (width 0.4064) (layer F.Cu) (net 19))
-  (segment (start 145.5928 108.7928) (end 145.5928 113.792) (width 0.4064) (layer F.Cu) (net 19))
-  (segment (start 118.620007 106.78) (end 134.42 106.78) (width 0.4064) (layer F.Cu) (net 19))
-  (segment (start 136.4 104.8) (end 141.6 104.8) (width 0.4064) (layer F.Cu) (net 19))
-  (segment (start 134.42 106.78) (end 136.4 104.8) (width 0.4064) (layer F.Cu) (net 19))
-  (segment (start 141.6 104.8) (end 145.5928 108.7928) (width 0.4064) (layer F.Cu) (net 19))
   (segment (start 142.8496 116.5352) (end 129.032 116.5352) (width 0.4064) (layer F.Cu) (net 19))
   (segment (start 129.032 116.5352) (end 127.2032 118.364) (width 0.4064) (layer F.Cu) (net 19))
@@
   (segment (start 242.1203 108.9903) (end 239.91 106.78) (width 0.4064) (layer B.Cu) (net 50))
   (segment (start 242.1203 111.196) (end 242.1203 108.9903) (width 0.4064) (layer B.Cu) (net 50))
-  (segment (start 135.114007 94.096) (end 124.970007 104.24) (width 0.4064) (layer B.Cu) (net 51))
-  (segment (start 162.5203 94.096) (end 135.114007 94.096) (width 0.4064) (layer B.Cu) (net 51))
+  (segment (start 162.5203 94.096) (end 137.031773 94.096) (width 0.4064) (layer B.Cu) (net 51))
+  (segment (start 126.887773 104.24) (end 126.808484 104.24) (width 0.4064) (layer B.Cu) (net 51))
+  (segment (start 137.031773 94.096) (end 126.887773 104.24) (width 0.4064) (layer B.Cu) (net 51))
+  (segment (start 126.808484 104.24) (end 124.970007 104.24) (width 0.4064) (layer B.Cu) (net 51))
+  (segment (start 123.660007 105.7) (end 123.660007 105.55) (width 0.4064) (layer B.Cu) (net 51))
+  (segment (start 123.660007 105.55) (end 124.970007 104.24) (width 0.4064) (layer B.Cu) (net 51))
   (segment (start 164.4203 92.196) (end 162.5203 94.096) (width 0.4064) (layer B.Cu) (net 51))
   (segment (start 134.5293 123.2593) (end 134.51 123.24) (width 0.4064) (layer B.Cu) (net 52))
